File: Carte_Drone/Carte_Drone.kicad_pcb (KiCad board)
At the start: 2 copper layers, 41.5 x 55 mm, 4 parts

Commit message: Changement typon et empreinte
Routing:
- net /RXB: track 21.9 -> 22.8 mm
Changed lines of the file:
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@@
 			(at 7.62 -17.78)
 			(size 2 2)
-			(drill 1.02)
+			(drill 0.8)
 			(layers "*.Cu" "*.Mask")
 			(remove_unused_layers no)
@@
 			(at 7.62 -15.24)
 			(size 2 2)
-			(drill 1.02)
+			(drill 0.8)
 			(layers "*.Cu" "*.Mask")
 			(remove_unused_layers no)
@@
 			(at 7.62 -12.7)
 			(size 2 2)
-			(drill 1.02)
+			(drill 0.8)
 			(layers "*.Cu" "*.Mask")
 			(remove_unused_layers no)
@@
 			(at 7.62 -10.16)
 			(size 2 2)
-			(drill 1.02)
+			(drill 0.8)
 			(layers "*.Cu" "*.Mask")
 			(remove_unused_layers no)
@@
 			(at 7.62 -7.62)
 			(size 2 2)
-			(drill 1.02)
+			(drill 0.8)
 			(layers "*.Cu" "*.Mask")
 			(remove_unused_layers no)
@@
 			(at 7.62 -5.08)
 			(size 2 2)
-			(drill 1.02)
+			(drill 0.8)
 			(layers "*.Cu" "*.Mask")
 			(remove_unused_layers no)
@@
 			(at 7.62 -2.54)
 			(size 2 2)
-			(drill 1.02)
+			(drill 0.8)
 			(layers "*.Cu" "*.Mask")
 			(remove_unused_layers no)
@@
 			(at 7.62 0)
 			(size 2 2)
-			(drill 1.02)
+			(drill 0.8)
 			(layers "*.Cu" "*.Mask")
 			(remove_unused_layers no)
@@
 			(at 7.62 2.54)
 			(size 2 2)
-			(drill 1.02)
+			(drill 0.8)
 			(layers "*.Cu" "*.Mask")
 			(remove_unused_layers no)
@@
 			(at 7.62 5.08)
 			(size 2 2)
-			(drill 1.02)
+			(drill 0.8)
 			(layers "*.Cu" "*.Mask")
 			(remove_unused_layers no)
@@
 			(at 7.62 7.62)
 			(size 2 2)
-			(drill 1.02)
+			(drill 0.8)
 			(layers "*.Cu" "*.Mask")
 			(remove_unused_layers no)
@@
 			(at 7.62 10.16)
 			(size 2 2)
-			(drill 1.02)
+			(drill 0.8)
 			(layers "*.Cu" "*.Mask")
 			(remove_unused_layers no)
@@
 			(at 7.62 12.7)
 			(size 2 2)
-			(drill 1.02)
+			(drill 0.8)
 			(layers "*.Cu" "*.Mask")
 			(remove_unused_layers no)
@@
 			(at 7.62 15.24)
 			(size 2 2)
-			(drill 1.02)
+			(drill 0.8)
 			(layers "*.Cu" "*.Mask")
 			(remove_unused_layers no)
@@
 			(at 7.62 17.78)
 			(size 2 2)
-			(drill 1.02)
+			(drill 0.8)
 			(layers "*.Cu" "*.Mask")
 			(remove_unused_layers no)
@@
 			(at -7.62 17.78)
 			(size 2 2)
-			(drill 1.02)
+			(drill 0.8)
 			(layers "*.Cu" "*.Mask")
 			(remove_unused_layers no)
@@
 			(at -7.62 15.24)
 			(size 2 2)
-			(drill 1.02)
+			(drill 0.8)
 			(layers "*.Cu" "*.Mask")
 			(remove_unused_layers no)
@@
 			(at -7.62 12.7)
 			(size 2 2)
-			(drill 1.02)
+			(drill 0.8)
 			(layers "*.Cu" "*.Mask")
 			(remove_unused_layers no)
@@
 			(at -7.62 10.16)
 			(size 2 2)
-			(drill 1.02)
+			(drill 0.8)
 			(layers "*.Cu" "*.Mask")
 			(remove_unused_layers no)
@@
 			(at -7.62 7.62)
 			(size 2 2)
-			(drill 1.02)
+			(drill 0.8)
 			(layers "*.Cu" "*.Mask")
 			(remove_unused_layers no)
@@
 			(at -7.62 5.08)
 			(size 2 2)
-			(drill 1.02)
+			(drill 0.8)
 			(layers "*.Cu" "*.Mask")
 			(remove_unused_layers no)
@@
 			(at -7.62 2.54)
 			(size 2 2)
-			(drill 1.02)
+			(drill 0.8)
 			(layers "*.Cu" "*.Mask")
 			(remove_unused_layers no)
@@
 			(at -7.62 0)
 			(size 2 2)
-			(drill 1.02)
+			(drill 0.8)
 			(layers "*.Cu" "*.Mask")
 			(remove_unused_layers no)
@@
 			(at -7.62 -2.54)
 			(size 2 2)
-			(drill 1.02)
+			(drill 0.8)
 			(layers "*.Cu" "*.Mask")
 			(remove_unused_layers no)
@@
 			(at -7.62 -5.08)
 			(size 2 2)
-			(drill 1.02)
+			(drill 0.8)
 			(layers "*.Cu" "*.Mask")
 			(remove_unused_layers no)
@@
 			(at -7.62 -7.62)
 			(size 2 2)
-			(drill 1.02)
+			(drill 0.8)
 			(layers "*.Cu" "*.Mask")
 			(remove_unused_layers no)
@@
 			(at -7.62 -10.16)
 			(size 2 2)
-			(drill 1.02)
+			(drill 0.8)
 			(layers "*.Cu" "*.Mask")
 			(remove_unused_layers no)
@@
 			(at -7.62 -12.7)
 			(size 2 2)
-			(drill 1.02)
+			(drill 0.8)
 			(layers "*.Cu" "*.Mask")
 			(remove_unused_layers no)
@@
 			(at -7.62 -15.24)
 			(size 2 2)
-			(drill 1.02)
+			(drill 0.8)
 			(layers "*.Cu" "*.Mask")
 			(remove_unused_layers no)
@@
 			(at -7.62 -17.78)
 			(size 2 2)
-			(drill 1.02)
+			(drill 0.8)
 			(layers "*.Cu" "*.Mask")
 			(remove_unused_layers no)
@@
 			(at 2.76 -1.8)
 			(size 2 2)
-			(drill 1.02)
+			(drill 0.8)
 			(layers "*.Cu" "*.Mask")
 			(remove_unused_layers no)
@@
 			(at 2.76 0.74)
 			(size 2 2)
-			(drill 1.02)
+			(drill 0.8)
 			(layers "*.Cu" "*.Mask")
 			(remove_unused_layers no)
@@
 			(at 2.76 3.28)
 			(size 2 2)
-			(drill 1.02)
+			(drill 0.8)
 			(layers "*.Cu" "*.Mask")
 			(remove_unused_layers no)
@@
 			(at 2.76 5.82)
 			(size 2 2)
-			(drill 1.02)
+			(drill 0.8)
 			(layers "*.Cu" "*.Mask")
 			(remove_unused_layers no)
@@
 			(at 2.76 8.36)
 			(size 2 2)
-			(drill 1.02)
+			(drill 0.8)
 			(layers "*.Cu" "*.Mask")
 			(remove_unused_layers no)
@@
 			(at 2.76 10.9)
 			(size 2 2)
-			(drill 1.02)
+			(drill 0.8)
 			(layers "*.Cu" "*.Mask")
 			(remove_unused_layers no)
@@
 			(at 2.66 0)
 			(size 2 2)
-			(drill 1.02)
+			(drill 0.8)
 			(layers "*.Cu" "*.Mask")
 			(remove_unused_layers no)
@@
 			(at 2.66 2.54)
 			(size 2 2)
-			(drill 1.02)
+			(drill 0.8)
 			(layers "*.Cu" "*.Mask")
 			(remove_unused_layers no)
@@
 			(at 2.66 5.08)
 			(size 2 2)
-			(drill 1.02)
+			(drill 0.8)
 			(layers "*.Cu" "*.Mask")
 			(remove_unused_layers no)
@@
 			(at 2.76 -1.8)
 			(size 2 2)
-			(drill 1.02)
+			(drill 0.8)
 			(layers "*.Cu" "*.Mask")
 			(remove_unused_layers no)
@@
 			(at 2.76 0.74)
 			(size 2 2)
-			(drill 1.02)
+			(drill 0.8)
 			(layers "*.Cu" "*.Mask")
 			(remove_unused_layers no)
@@
 			(at 2.76 3.28)
 			(size 2 2)
-			(drill 1.02)
+			(drill 0.8)
 			(layers "*.Cu" "*.Mask")
 			(remove_unused_layers no)
@@
 			(at 2.76 5.82)
 			(size 2 2)
-			(drill 1.02)
+			(drill 0.8)
 			(layers "*.Cu" "*.Mask")
 			(remove_unused_layers no)
@@
 			(at 2.76 8.36)
 			(size 2 2)
-			(drill 1.02)
+			(drill 0.8)
 			(layers "*.Cu" "*.Mask")
 			(remove_unused_layers no)
@@
 			(at 2.76 10.9)
 			(size 2 2)
-			(drill 1.02)
+			(drill 0.8)
 			(layers "*.Cu" "*.Mask")
 			(remove_unused_layers no)
@@
 	)
 	(segment
-		(start 203 80.6)
-		(end 203.8 79.8)
+		(start 203 79.1)
+		(end 203 92.6)
 		(width 0.5)
 		(layer "B.Cu")
@@
 	)
 	(segment
+		(start 201.84 93.76)
+		(end 197.79 93.76)
+		(width 0.5)
+		(layer "B.Cu")
+		(net 31)
+	)
+	(segment
+		(start 203.82 78.28)
+		(end 203 79.1)
+		(width 0.5)
+		(layer "B.Cu")
+		(net 31)
+	)
+	(segment
+		(start 206.26 78.28)
+		(end 203.82 78.28)
+		(width 0.5)
+		(layer "B.Cu")
+		(net 31)
+	)
+	(segment
 		(start 203 92.6)
-		(end 203 80.6)
-		(width 0.5)
-		(layer "B.Cu")
-		(net 31)
-	)
-	(segment
-		(start 203.8 79.8)
-		(end 204.74 79.8)
-		(width 0.5)
-		(layer "B.Cu")
-		(net 31)
-	)
-	(segment
-		(start 204.74 79.8)
-		(end 206.26 78.28)
-		(width 0.5)
-		(layer "B.Cu")
-		(net 31)
-	)
-	(segment
-		(start 197.79 93.76)
 		(end 201.84 93.76)
-		(width 0.5)
-		(layer "B.Cu")
-		(net 31)
-	)
-	(segment
-		(start 201.84 93.76)
-		(end 203 92.6)
 		(width 0.5)
 		(layer "B.Cu")
@@
 			(clearance 0.7)
 		)
-		(min_thickness 0.5)
+		(min_thickness 0.25)
 		(filled_areas_thickness no)
 		(fill yes

Commit message: modif typon 2 création Sysml
Connections:
- U1 pad 15: unconnected-(U1-D13-Pad15) -> /RXB
- U1 pad 16: unconnected-(U1-D12-Pad16) -> /TXB
- U1 pad 23: /RXB -> unconnected-(U1-D5-Pad23)
- U1 pad 24: /TXB -> unconnected-(U1-D4-Pad24)
Routing:
- net /3V3: track 84.8 -> 103.7 mm
- net /TXB: track 22.6 -> 10.5 mm
- net /RXB: track 22.8 -> 27.2 mm
Changed lines of the file:
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@@
 	(net 11 "unconnected-(U1-+5V-Pad4)")
 	(net 12 "unconnected-(U1-NRST-Pad3)")
-	(net 13 "unconnected-(U1-D13-Pad15)")
+	(net 13 "unconnected-(U1-D5-Pad23)")
 	(net 14 "unconnected-(U1-A7-Pad5)")
-	(net 15 "unconnected-(U1-D12-Pad16)")
+	(net 15 "unconnected-(U1-D4-Pad24)")
 	(net 16 "unconnected-(U1-D7-Pad21)")
 	(net 17 "unconnected-(U1-D6-Pad22)")
@@
 			(layers "*.Cu" "*.Mask")
 			(remove_unused_layers no)
-			(net 13 "unconnected-(U1-D13-Pad15)")
+			(net 31 "/RXB")
 			(pinfunction "D13")
 			(pintype "bidirectional")
@@
 			(layers "*.Cu" "*.Mask")
 			(remove_unused_layers no)
-			(net 15 "unconnected-(U1-D12-Pad16)")
+			(net 30 "/TXB")
 			(pinfunction "D12")
 			(pintype "bidirectional")
@@
 			(layers "*.Cu" "*.Mask")
 			(remove_unused_layers no)
-			(net 31 "/RXB")
+			(net 13 "unconnected-(U1-D5-Pad23)")
 			(pinfunction "D5")
 			(pintype "bidirectional")
@@
 			(layers "*.Cu" "*.Mask")
 			(remove_unused_layers no)
-			(net 30 "/TXB")
+			(net 15 "unconnected-(U1-D4-Pad24)")
 			(pinfunction "D4")
 			(pintype "bidirectional")
@@
 	)
 	(segment
-		(start 221.5 93.52)
-		(end 213.42 101.6)
+		(start 197 101.6)
+		(end 233.3 101.6)
 		(width 0.5)
 		(layer "B.Cu")
@@
 	)
 	(segment
+		(start 233.3 101.6)
+		(end 234.85 100.05)
+		(width 0.5)
+		(layer "B.Cu")
+		(net 2)
+	)
+	(segment
 		(start 233.08 93.52)
-		(end 235.249 91.351)
+		(end 234.85 91.75)
 		(width 0.5)
 		(layer "B.Cu")
@@
 	)
 	(segment
+		(start 234.85 91.75)
+		(end 235.249 91.351)
+		(width 0.5)
+		(layer "B.Cu")
+		(net 2)
+	)
+	(segment
 		(start 235.249 91.351)
 		(end 235.249 81.4)
@@
 	)
 	(segment
-		(start 213.42 101.6)
-		(end 197 101.6)
-		(width 0.5)
-		(layer "B.Cu")
-		(net 2)
-	)
-	(segment
 		(start 197 101.6)
 		(end 195.4 100)
@@
 	)
 	(segment
+		(start 234.85 100.05)
+		(end 234.85 91.75)
+		(width 0.5)
+		(layer "B.Cu")
+		(net 2)
+	)
+	(segment
 		(start 197.79 86.14)
 		(end 196.66 86.14)
@@
 	)
 	(segment
-		(start 202.86 75.74)
-		(end 206.26 75.74)
+		(start 202.64 96.06)
+		(end 206.26 96.06)
 		(width 0.5)
 		(layer "B.Cu")
@@
 	)
 	(segment
-		(start 201.6 90.2)
-		(end 201.6 77)
+		(start 197.8 91.22)
+		(end 202.64 96.06)
 		(width 0.5)
 		(layer "B.Cu")
@@
 	)
 	(segment
-		(start 200.58 91.22)
-		(end 201.6 90.2)
-		(width 0.5)
-		(layer "B.Cu")
-		(net 30)
-	)
-	(segment
-		(start 197.79 91.22)
-		(end 200.58 91.22)
-		(width 0.5)
-		(layer "B.Cu")
-		(net 30)
-	)
-	(segment
-		(start 201.6 77)
-		(end 202.86 75.74)
-		(width 0.5)
-		(layer "B.Cu")
-		(net 30)
-	)
-	(segment
-		(start 203 79.1)
-		(end 203 92.6)
+		(start 218.46 99.1)
+		(end 221.5 96.06)
 		(width 0.5)
 		(layer "B.Cu")
@@
 	)
 	(segment
-		(start 201.84 93.76)
-		(end 197.79 93.76)
+		(start 203.14 99.1)
+		(end 218.46 99.1)
 		(width 0.5)
 		(layer "B.Cu")
@@
 	)
 	(segment
-		(start 203.82 78.28)
-		(end 203 79.1)
-		(width 0.5)
-		(layer "B.Cu")
-		(net 31)
-	)
-	(segment
-		(start 206.26 78.28)
-		(end 203.82 78.28)
-		(width 0.5)
-		(layer "B.Cu")
-		(net 31)
-	)
-	(segment
-		(start 203 92.6)
-		(end 201.84 93.76)
-		(width 0.5)
-		(layer "B.Cu")
+		(start 197.8 93.76)
+		(end 203.14 99.1)
+		(width 0.5)
+		(layer "B.Cu")
