File: Carte_Drone/Carte_Drone.kicad_sch (KiCad schematic)
At the start: 4 parts

Commit message: Changement empreinte 1
Parts:
- BLU1, GPS1: footprint Connector_PinSocket_1.27mm:PinSocket_1x06_P1.27mm_Vertical -> Librairie_Drone:PinSocket_1x06_P1.27mm_Vertical_2
- U3: footprint Connector_PinSocket_1.27mm:PinSocket_1x03_P1.27mm_Vertical -> Librairie_Drone:PinSocket_1x03_P1.27mm_Vertical_2
Changed lines of the file:
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@@
 	(wire
 		(pts
-			(xy 83.82 44.45) (xy 83.82 45.72)
-		)
-		(stroke
-			(width 0)
-			(type default)
-		)
-	)
-	(wire
-		(pts
-			(xy 71.12 59.69) (xy 77.47 59.69)
+			(xy 71.12 59.69) (xy 74.93 59.69)
 		)
 		(stroke
@@
 	(wire
 		(pts
-			(xy 97.79 44.45) (xy 105.41 44.45)
+			(xy 101.6 44.45) (xy 105.41 44.45)
 		)
 		(stroke
@@
 	(wire
 		(pts
-			(xy 100.33 52.07) (xy 106.68 52.07)
+			(xy 100.33 52.07) (xy 101.6 52.07)
 		)
 		(stroke
@@
 	(wire
 		(pts
-			(xy 85.09 54.61) (xy 88.9 54.61)
+			(xy 86.36 54.61) (xy 88.9 54.61)
 		)
 		(stroke
@@
 	(wire
 		(pts
-			(xy 106.68 52.07) (xy 106.68 53.34)
-		)
-		(stroke
-			(width 0)
-			(type default)
-		)
-	)
-	(wire
-		(pts
-			(xy 77.47 44.45) (xy 83.82 44.45)
+			(xy 77.47 44.45) (xy 80.01 44.45)
 		)
 		(stroke
@@
 	(wire
 		(pts
-			(xy 85.09 55.88) (xy 85.09 54.61)
-		)
-		(stroke
-			(width 0)
-			(type default)
-		)
-	)
-	(wire
-		(pts
 			(xy 86.36 52.07) (xy 88.9 52.07)
-		)
-		(stroke
-			(width 0)
-			(type default)
-		)
-	)
-	(wire
-		(pts
-			(xy 77.47 59.69) (xy 77.47 64.77)
 		)
 		(stroke
@@
 	(symbol
 		(lib_id "power:Earth")
-		(at 85.09 55.88 0)
+		(at 86.36 54.61 270)
 		(unit 1)
 		(exclude_from_sim no)
@@
 		(on_board yes)
 		(dnp no)
-		(fields_autoplaced yes)
 		(property "Reference" "#PWR03"
-			(at 85.09 62.23 0)
+			(at 80.01 54.61 0)
 			(effects
 				(font
@@
 		)
 		(property "Value" "Earth"
-			(at 85.09 60.96 0)
+			(at 81.026 54.61 90)
 			(effects
 				(font
@@
 		)
 		(property "Footprint" ""
-			(at 85.09 55.88 0)
+			(at 86.36 54.61 0)
 			(effects
 				(font
@@
 		)
 		(property "Datasheet" "~"
-			(at 85.09 55.88 0)
+			(at 86.36 54.61 0)
 			(effects
 				(font
@@
 		)
 		(property "Description" "Power symbol creates a global label with name \"Earth\""
-			(at 85.09 55.88 0)
+			(at 86.36 54.61 0)
 			(effects
 				(font
@@
 	(symbol
 		(lib_id "power:Earth")
-		(at 97.79 44.45 0)
+		(at 101.6 44.45 270)
 		(unit 1)
 		(exclude_from_sim no)
@@
 		(dnp no)
 		(property "Reference" "#PWR05"
-			(at 97.79 50.8 0)
+			(at 95.25 44.45 0)
 			(effects
 				(font
@@
 		)
 		(property "Value" "Earth"
-			(at 97.79 48.26 0)
+			(at 96.266 44.45 90)
 			(effects
 				(font
@@
 		)
 		(property "Footprint" ""
-			(at 97.79 44.45 0)
+			(at 101.6 44.45 0)
 			(effects
 				(font
@@
 		)
 		(property "Datasheet" "~"
-			(at 97.79 44.45 0)
+			(at 101.6 44.45 0)
 			(effects
 				(font
@@
 		)
 		(property "Description" "Power symbol creates a global label with name \"Earth\""
-			(at 97.79 44.45 0)
+			(at 101.6 44.45 0)
 			(effects
 				(font
@@
 			)
 		)
-		(property "Footprint" "Connector_PinSocket_1.27mm:PinSocket_1x03_P1.27mm_Vertical"
+		(property "Footprint" "Librairie_Drone:PinSocket_1x03_P1.27mm_Vertical_2"
 			(at 69.85 41.91 0)
 			(effects
@@
 			)
 		)
-		(property "Footprint" "Connector_PinSocket_1.27mm:PinSocket_1x06_P1.27mm_Vertical"
+		(property "Footprint" "Librairie_Drone:PinSocket_1x06_P1.27mm_Vertical_2"
 			(at 109.22 39.37 0)
 			(effects
@@
 	(symbol
 		(lib_id "power:Earth")
-		(at 106.68 53.34 0)
+		(at 101.6 52.07 90)
 		(unit 1)
 		(exclude_from_sim no)
@@
 		(fields_autoplaced yes)
 		(property "Reference" "#PWR01"
-			(at 106.68 59.69 0)
+			(at 107.95 52.07 0)
 			(effects
 				(font
@@
 		)
 		(property "Value" "Earth"
-			(at 106.68 58.42 0)
-			(effects
-				(font
-					(size 1.27 1.27)
-				)
+			(at 105.41 52.0699 90)
+			(effects
+				(font
+					(size 1.27 1.27)
+				)
+				(justify right)
 			)
 		)
 		(property "Footprint" ""
-			(at 106.68 53.34 0)
+			(at 101.6 52.07 0)
 			(effects
 				(font
@@
 		)
 		(property "Datasheet" "~"
-			(at 106.68 53.34 0)
+			(at 101.6 52.07 0)
 			(effects
 				(font
@@
 		)
 		(property "Description" "Power symbol creates a global label with name \"Earth\""
-			(at 106.68 53.34 0)
+			(at 101.6 52.07 0)
 			(effects
 				(font
@@
 	(symbol
 		(lib_id "power:Earth")
-		(at 83.82 45.72 0)
+		(at 80.01 44.45 90)
 		(unit 1)
 		(exclude_from_sim no)
@@
 		(on_board yes)
 		(dnp no)
-		(fields_autoplaced yes)
 		(property "Reference" "#PWR04"
-			(at 83.82 52.07 0)
+			(at 86.36 44.45 0)
 			(effects
 				(font
@@
 		)
 		(property "Value" "Earth"
-			(at 83.82 50.8 0)
-			(effects
-				(font
-					(size 1.27 1.27)
-				)
+			(at 82.804 44.45 90)
+			(effects
+				(font
+					(size 1.27 1.27)
+				)
+				(justify right)
 			)
 		)
 		(property "Footprint" ""
-			(at 83.82 45.72 0)
+			(at 80.01 44.45 0)
 			(effects
 				(font
@@
 		)
 		(property "Datasheet" "~"
-			(at 83.82 45.72 0)
+			(at 80.01 44.45 0)
 			(effects
 				(font
@@
 		)
 		(property "Description" "Power symbol creates a global label with name \"Earth\""
-			(at 83.82 45.72 0)
+			(at 80.01 44.45 0)
 			(effects
 				(font
@@
 	(symbol
 		(lib_id "power:Earth")
-		(at 77.47 64.77 0)
+		(at 74.93 59.69 90)
 		(unit 1)
 		(exclude_from_sim no)
@@
 		(on_board yes)
 		(dnp no)
-		(fields_autoplaced yes)
 		(property "Reference" "#PWR02"
-			(at 77.47 71.12 0)
+			(at 81.28 59.69 0)
 			(effects
 				(font
@@
 		)
 		(property "Value" "Earth"
-			(at 77.47 69.85 0)
-			(effects
-				(font
-					(size 1.27 1.27)
-				)
+			(at 77.47 59.69 90)
+			(effects
+				(font
+					(size 1.27 1.27)
+				)
+				(justify right)
 			)
 		)
 		(property "Footprint" ""
-			(at 77.47 64.77 0)
+			(at 74.93 59.69 0)
 			(effects
 				(font
@@
 		)
 		(property "Datasheet" "~"
-			(at 77.47 64.77 0)
+			(at 74.93 59.69 0)
 			(effects
 				(font
@@
 		)
 		(property "Description" "Power symbol creates a global label with name \"Earth\""
-			(at 77.47 64.77 0)
+			(at 74.93 59.69 0)
 			(effects
 				(font
@@
 			)
 		)
-		(property "Footprint" "Connector_PinSocket_1.27mm:PinSocket_1x06_P1.27mm_Vertical"
+		(property "Footprint" "Librairie_Drone:PinSocket_1x06_P1.27mm_Vertical_2"
 			(at 66.04 52.07 0)
 			(effects

Commit message: modif typon 2 création Sysml
Connections:
- net RXB: now also U1.15 (D13); no longer U1.23 (D5)
- net TXB: now also U1.16 (D12); no longer U1.24 (D4)
Changed lines of the file:
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@@
-	(wire
-		(pts
-			(xy 86.36 59.69) (xy 88.9 59.69)
-		)
-		(stroke
-			(width 0)
-			(type default)
-		)
-	)
 	(wire
 		(pts
@@
 	(wire
 		(pts
-			(xy 86.36 58.42) (xy 88.9 58.42)
-		)
-		(stroke
-			(width 0)
-			(type default)
-		)
-	)
-	(wire
-		(pts
 			(xy 100.33 52.07) (xy 101.6 52.07)
 		)
@@
 	(wire
 		(pts
+			(xy 86.36 68.58) (xy 88.9 68.58)
+		)
+		(stroke
+			(width 0)
+			(type default)
+		)
+	)
+	(wire
+		(pts
 			(xy 77.47 46.99) (xy 80.01 46.99)
 		)
@@
 		(pts
 			(xy 86.36 52.07) (xy 88.9 52.07)
+		)
+		(stroke
+			(width 0)
+			(type default)
+		)
+	)
+	(wire
+		(pts
+			(xy 100.33 68.58) (xy 104.14 68.58)
 		)
 		(stroke
@@
 		)
 	)
+	(label "RXB"
+		(at 101.6 68.58 0)
+		(effects
+			(font
+				(size 0.508 0.508)
+			)
+			(justify left bottom)
+		)
+	)
 	(label "3V3"
 		(at 77.47 45.72 0)
@@
 	)
 	(label "TXB"
-		(at 87.63 58.42 0)
-		(effects
-			(font
-				(size 0.508 0.508)
-			)
-			(justify left bottom)
-		)
-	)
-	(label "RXB"
-		(at 87.63 59.69 0)
-		(effects
-			(font
+		(at 87.63 68.58 0)
+		(effects
+			(font
